Commit message: Francis model update

File: walkTraining/plane.urdf (robot description, URDF)
Before this commit: robot plane, 1 links, 0 joints
Links:
- link planeLink: geometry collision box size=30 30 0.001; visual box size=30 30 0.001

File: walkTraining/test.urdf (robot description, URDF)
Before this commit: robot plane, 1 links, 0 joints
Links:
- removed link planeLink
- added link body, mass .0; visual cylinder length=0.05 radius=0.375
- added link leg1_top_shoulder1, mass .0; visual sphere radius=0.07
Joints:
- added joint leg1_top_articulation1: type revolute, parent body, child leg1_top_shoulder1, origin xyz=0.375 0 1 rpy=0 0 0, axis 0 0 1, limit lower=-2 upper=2 effort=30 velocity=1.0
